File: design_files/greenhouse.kicad_sch (KiCad schematic)
At the start: 7 parts, among them M1 Fan_3pin, U1 SensorSoilMoisture, U4 LM35-D

Commit message: updated kicad scheme
a wire was omitted
Connections:
- net at RM1.3 (IN): now also A1.22 (GP17)
Changed lines of the file:
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@@
+	(wire
+		(pts
+			(xy 172.72 35.56) (xy 185.42 35.56)
+		)
+		(stroke
+			(width 0)
+			(type default)
+		)
+	)
 	(wire
 		(pts
@@
 	(wire
 		(pts
+			(xy 185.42 35.56) (xy 185.42 114.3)
+		)
+		(stroke
+			(width 0)
+			(type default)
+		)
+	)
+	(wire
+		(pts
 			(xy 176.53 93.98) (xy 215.9 93.98)
 		)
@@
 		)
 		(stroke
+			(width 0)
+			(type default)
+		)
+	)
+	(wire
+		(pts
+			(xy 185.42 114.3) (xy 176.53 114.3)
+		)
+		(stroke
